Commit message: locate me review correction

File: Projects/LocateMe/catkin_ws/src/my_robot/urdf/my_robot.xacro (robot description, xacro)
@@ -4,5 +4,5 @@
     <link name="robot_footprint"></link>
     <joint name="robot_footprint_joint" type="fixed">
-        <origin xyz="0 0 0" rpy="0 0 0" />
+        <origin xyz="0 0 0.1" rpy="0 0 0" />
         <parent link="robot_footprint"/>
         <child link="chassis" />
